File: sa2011_mic_amp.kicad_pcb (KiCad board)
At the start: 2 copper layers, 23.1 x 37.1 mm, 12 parts, among them J2 Conn_01x02_Pin, SW1 SW_SPST, U1 SA2011

Commit message: 配置を修正
Parts:
- R3: footprint Resistor_THT:R_Axial_DIN0207_L6.3mm_D2.5mm_P2.54mm_Vertical -> Resistor_THT:R_Axial_DIN0207_L6.3mm_D2.5mm_P7.62mm_Horizontal
- moved R3 6.23 mm to (164.1, 99.5), turned to 180 degrees
- moved C6 2.35 mm to (157.5, 95.0), turned to 0 degrees
- moved SW1 1.00 mm to (152.4, 95.5), turned to 90 degrees
- moved J2 0.62 mm to (163.1, 88.8)
- moved C1 0.06 mm to (151.3, 88.1)
Routing:
- net VCC 4～14v: track 36.9 -> 30.0 mm
- net Net-(SW1-B): track 11.0 -> 4.71 mm
- net GND: track 75.0 -> 77.0 mm
